Commit message: proper robot description package

File: cat_packages/jb2a_description/urdf/jb2a.urdf.xacro (robot description, xacro)
@@ -52,5 +52,5 @@
     <visual>
       <geometry>
-        <mesh filename="package://my_urdf_tutorial/meshes/base.stl"/>
+        <mesh filename="package://jb2a_description/meshes/base.stl"/>
       </geometry>
       <material name="gray"/>
@@ -61,5 +61,5 @@
     <visual>
       <geometry>
-        <mesh filename="package://my_urdf_tutorial/meshes/bearings.stl"/>
+        <mesh filename="package://jb2a_description/meshes/bearings.stl"/>
       </geometry>
       <material name="black"/>
@@ -75,5 +75,5 @@
     <visual>
       <geometry>
-        <mesh filename="package://my_urdf_tutorial/meshes/bearings.stl"/>
+        <mesh filename="package://jb2a_description/meshes/bearings.stl"/>
       </geometry>
       <material name="black"/>
@@ -90,5 +90,5 @@
     <visual>
       <geometry>
-        <mesh filename="package://my_urdf_tutorial/meshes/Piece100.stl"/>
+        <mesh filename="package://jb2a_description/meshes/Piece100.stl"/>
       </geometry>
       <material name="gray"/>
@@ -106,5 +106,5 @@
     <visual>
       <geometry>
-        <mesh filename="package://my_urdf_tutorial/meshes/Piece11.stl"/>
+        <mesh filename="package://jb2a_description/meshes/Piece11.stl"/>
       </geometry>
       <material name="gray"/>
@@ -120,5 +120,5 @@
     <visual>
       <geometry>
-        <mesh filename="package://my_urdf_tutorial/meshes/Piece11sym.stl"/>
+        <mesh filename="package://jb2a_description/meshes/Piece11sym.stl"/>
       </geometry>
       <material name="gray"/>
@@ -135,5 +135,5 @@
     <visual>
       <geometry>
-        <mesh filename="package://my_urdf_tutorial/meshes/arm1-Piece12.stl"/>
+        <mesh filename="package://jb2a_description/meshes/arm1-Piece12.stl"/>
       </geometry>
       <material name="green"/>
@@ -151,5 +151,5 @@
     <visual>
       <geometry>
-        <mesh filename="package://my_urdf_tutorial/meshes/arm1-Piece15.stl"/>
+        <mesh filename="package://jb2a_description/meshes/arm1-Piece15.stl"/>
       </geometry>
       <material name="cyan"/>
@@ -167,5 +167,5 @@
     <visual>
       <geometry>
-        <mesh filename="package://my_urdf_tutorial/meshes/arm1-Piece13.stl"/>
+        <mesh filename="package://jb2a_description/meshes/arm1-Piece13.stl"/>
       </geometry>
       <material name="red"/>
@@ -181,5 +181,5 @@
     <visual>
       <geometry>
-        <mesh filename="package://my_urdf_tutorial/meshes/arm1-Piece13.stl"/>
+        <mesh filename="package://jb2a_description/meshes/arm1-Piece13.stl"/>
       </geometry>
       <material name="red"/>
@@ -195,5 +195,5 @@
     <visual>
       <geometry>
-        <mesh filename="package://my_urdf_tutorial/meshes/arm1-Piece13.stl"/>
+        <mesh filename="package://jb2a_description/meshes/arm1-Piece13.stl"/>
       </geometry>
       <material name="red"/>
@@ -210,5 +210,5 @@
     <visual>
       <geometry>
-        <mesh filename="package://my_urdf_tutorial/meshes/arm2-Piece16.stl"/>
+        <mesh filename="package://jb2a_description/meshes/arm2-Piece16.stl"/>
       </geometry>
       <material name="pink"/>
@@ -226,5 +226,5 @@
     <visual>
       <geometry>
-        <mesh filename="package://my_urdf_tutorial/meshes/arm2-Piece17.stl"/>
+        <mesh filename="package://jb2a_description/meshes/arm2-Piece17.stl"/>
       </geometry>
       <material name="red"/>
@@ -240,5 +240,5 @@
     <visual>
       <geometry>
-        <mesh filename="package://my_urdf_tutorial/meshes/arm2-Piece17.stl"/>
+        <mesh filename="package://jb2a_description/meshes/arm2-Piece17.stl"/>
       </geometry>
       <material name="red"/>
@@ -254,5 +254,5 @@
     <visual>
       <geometry>
-        <mesh filename="package://my_urdf_tutorial/meshes/arm2-Piece14.stl"/>
+        <mesh filename="package://jb2a_description/meshes/arm2-Piece14.stl"/>
       </geometry>
       <material name="turcoise"/>
@@ -269,5 +269,5 @@
     <visual>
       <geometry>
-        <mesh filename="package://my_urdf_tutorial/meshes/arm3-Piece17.stl"/>
+        <mesh filename="package://jb2a_description/meshes/arm3-Piece17.stl"/>
       </geometry>
       <material name="pink_light"/>
@@ -285,5 +285,5 @@
     <visual>
       <geometry>
-        <mesh filename="package://my_urdf_tutorial/meshes/arm3-Piece18.stl"/>
+        <mesh filename="package://jb2a_description/meshes/arm3-Piece18.stl"/>
       </geometry>
       <material name="cyan_light"/>
@@ -299,5 +299,5 @@
     <visual>
       <geometry>
-        <mesh filename="package://my_urdf_tutorial/meshes/arm3-Piece19.stl"/>
+        <mesh filename="package://jb2a_description/meshes/arm3-Piece19.stl"/>
       </geometry>
       <material name="red_light"/>
